File: necpc8801typea.kicad_sch (KiCad schematic)
At the start: 265 parts, among them J1 Conn_01x01, J2 Conn_01x06, J4 Conn_01x04, Q1 Q_PMOS_GSD AO3401A, Q2 Q_NMOS_GSD 2N7002, Q3 Q_NMOS_GSD 2N7002, SW1 SW_Push, U1 AMS1117-3.3, U2 TPS2553DBVR, U3 STM32F401RETx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

Commit message: updates
Connections:
- net +3.3VA: no longer R16.1, R17.1
- net GND: now also R16.1, R17.1
Changed lines of the file:
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@@
   (junction (at 121.92 26.67) (diameter 0) (color 0 0 0 0)
   )
+  (junction (at 73.66 158.75) (diameter 0) (color 0 0 0 0)
+  )
   (junction (at 213.36 107.315) (diameter 0) (color 0 0 0 0)
   )
@@
   (junction (at 91.44 243.84) (diameter 1.016) (color 0 0 0 0)
   )
+  (junction (at 73.66 147.32) (diameter 0) (color 0 0 0 0)
+  )
   (junction (at 330.2 273.05) (diameter 0) (color 0 0 0 0)
   )
@@
   (junction (at 233.68 281.94) (diameter 1.016) (color 0 0 0 0)
   )
+  (junction (at 73.66 139.7) (diameter 0) (color 0 0 0 0)
+  )
   (junction (at 127 243.84) (diameter 1.016) (color 0 0 0 0)
   )
@@
   (junction (at 57.15 243.84) (diameter 1.016) (color 0 0 0 0)
   )
+  (junction (at 73.66 143.51) (diameter 0) (color 0 0 0 0)
+  )
   (junction (at 278.13 311.15) (diameter 1.016) (color 0 0 0 0)
   )
@@
     (stroke (width 0) (type solid))
   )
+  (wire (pts (xy 73.66 137.16) (xy 73.66 139.7))
+    (stroke (width 0) (type default))
+  )
   (wire (pts (xy 337.82 300.99) (xy 337.82 320.04))
     (stroke (width 0) (type solid))
@@
     (stroke (width 0) (type solid))
   )
+  (wire (pts (xy 73.66 158.75) (xy 73.66 161.29))
+    (stroke (width 0) (type default))
+  )
   (wire (pts (xy 337.82 243.84) (xy 337.82 262.89))
     (stroke (width 0) (type solid))
@@
     (stroke (width 0) (type solid))
   )
+  (wire (pts (xy 73.66 154.94) (xy 73.66 158.75))
+    (stroke (width 0) (type default))
+  )
   (wire (pts (xy 19.685 26.67) (xy 22.86 26.67))
     (stroke (width 0) (type default))
@@
     (stroke (width 0) (type solid))
   )
+  (wire (pts (xy 73.66 143.51) (xy 73.66 147.32))
+    (stroke (width 0) (type default))
+  )
   (wire (pts (xy 171.45 306.07) (xy 173.99 306.07))
     (stroke (width 0) (type solid))
@@
     (stroke (width 0) (type solid))
   )
+  (wire (pts (xy 73.66 139.7) (xy 73.66 143.51))
+    (stroke (width 0) (type default))
+  )
   (wire (pts (xy 226.06 330.2) (xy 242.57 330.2))
     (stroke (width 0) (type solid))
@@
     (stroke (width 0) (type solid))
   )
+  (wire (pts (xy 73.66 147.32) (xy 73.66 151.13))
+    (stroke (width 0) (type default))
+  )
   (wire (pts (xy 355.6 300.99) (xy 355.6 281.94))
     (stroke (width 0) (type solid))
@@
     )
   )
-  (symbol (lib_id "controller-rescue:+3.3V-power") (at 73.66 147.32 270) (unit 1)
-    (in_bom yes) (on_board yes) (dnp no)
-    (property "Reference" "#PWR0118" (at 69.85 147.32 0)
-      (effects (font (size 1.27 1.27)) hide)
-    )
-    (property "Value" "+3.3V" (at 76.9112 147.701 90)
-      (effects (font (size 1.27 1.27)) (justify left))
-    )
-    (property "Footprint" "" (at 73.66 147.32 0)
-      (effects (font (size 1.27 1.27)) hide)
-    )
-    (property "Datasheet" "" (at 73.66 147.32 0)
-      (effects (font (size 1.27 1.27)) hide)
-    )
-    (pin "1")
-    (instances
-      (project "necpc8801typea"
-        (path "/151da08b-0979-4785-a9bf-6fa9b165d629"
-          (reference "#PWR0118") (unit 1)
-        )
-      )
-      (project "controller"
-        (path "/d7b41e20-3ed8-4e20-8d18-95c1ff55bd12"
-          (reference "#PWR0118") (unit 1)
-        )
-      )
-    )
-  )
   (symbol (lib_id "controller-rescue:GND-power") (at 52.07 94.615 0) (unit 1)
     (in_bom yes) (on_board yes) (dnp no)
@@
     )
   )
-  (symbol (lib_id "controller-rescue:+3.3V-power") (at 73.66 154.94 270) (unit 1)
-    (in_bom yes) (on_board yes) (dnp no)
-    (property "Reference" "#PWR0126" (at 69.85 154.94 0)
-      (effects (font (size 1.27 1.27)) hide)
-    )
-    (property "Value" "+3.3V" (at 76.9112 155.321 90)
-      (effects (font (size 1.27 1.27)) (justify left))
-    )
-    (property "Footprint" "" (at 73.66 154.94 0)
-      (effects (font (size 1.27 1.27)) hide)
-    )
-    (property "Datasheet" "" (at 73.66 154.94 0)
-      (effects (font (size 1.27 1.27)) hide)
-    )
-    (pin "1")
-    (instances
-      (project "necpc8801typea"
-        (path "/151da08b-0979-4785-a9bf-6fa9b165d629"
-          (reference "#PWR0126") (unit 1)
-        )
-      )
-      (project "controller"
-        (path "/d7b41e20-3ed8-4e20-8d18-95c1ff55bd12"
-          (reference "#PWR0105") (unit 1)
-        )
-      )
-    )
-  )
   (symbol (lib_id "MX_Alps_Hybrid:mx-alps-nec") (at 334.01 264.16 0) (unit 1)
     (in_bom yes) (on_board yes) (dnp no)
@@
     )
   )
-  (symbol (lib_id "controller-rescue:+3.3V-power") (at 73.66 158.75 270) (unit 1)
-    (in_bom yes) (on_board yes) (dnp no)
-    (property "Reference" "#PWR0127" (at 69.85 158.75 0)
-      (effects (font (size 1.27 1.27)) hide)
-    )
-    (property "Value" "+3.3V" (at 76.9112 159.131 90)
-      (effects (font (size 1.27 1.27)) (justify left))
-    )
-    (property "Footprint" "" (at 73.66 158.75 0)
-      (effects (font (size 1.27 1.27)) hide)
-    )
-    (property "Datasheet" "" (at 73.66 158.75 0)
-      (effects (font (size 1.27 1.27)) hide)
-    )
-    (pin "1")
-    (instances
-      (project "necpc8801typea"
-        (path "/151da08b-0979-4785-a9bf-6fa9b165d629"
-          (reference "#PWR0127") (unit 1)
-        )
-      )
-      (project "controller"
-        (path "/d7b41e20-3ed8-4e20-8d18-95c1ff55bd12"
-          (reference "#PWR0105") (unit 1)
-        )
-      )
-    )
-  )
   (symbol (lib_id "controller-rescue:GND-power") (at 99.06 94.615 0) (unit 1)
     (in_bom yes) (on_board yes) (dnp no)
@@
     )
   )
-  (symbol (lib_id "controller-rescue:+3.3V-power") (at 73.66 151.13 270) (unit 1)
-    (in_bom yes) (on_board yes) (dnp no)
-    (property "Reference" "#PWR0105" (at 69.85 151.13 0)
-      (effects (font (size 1.27 1.27)) hide)
-    )
-    (property "Value" "+3.3V" (at 76.9112 151.511 90)
-      (effects (font (size 1.27 1.27)) (justify left))
-    )
-    (property "Footprint" "" (at 73.66 151.13 0)
-      (effects (font (size 1.27 1.27)) hide)
-    )
-    (property "Datasheet" "" (at 73.66 151.13 0)
-      (effects (font (size 1.27 1.27)) hide)
-    )
-    (pin "1")
-    (instances
-      (project "necpc8801typea"
-        (path "/151da08b-0979-4785-a9bf-6fa9b165d629"
-          (reference "#PWR0105") (unit 1)
-        )
-      )
-      (project "controller"
-        (path "/d7b41e20-3ed8-4e20-8d18-95c1ff55bd12"
-          (reference "#PWR0105") (unit 1)
-        )
-      )
-    )
-  )
   (symbol (lib_id "Device:D_Small") (at 347.98 308.61 90) (unit 1)
     (in_bom yes) (on_board yes) (dnp no)
@@
     )
   )
-  (symbol (lib_id "controller-rescue:+3.3V-power") (at 73.66 139.7 270) (unit 1)
+  (symbol (lib_id "controller-rescue:+3.3V-power") (at 73.66 137.16 0) (unit 1)
     (in_bom yes) (on_board yes) (dnp no)
-    (property "Reference" "#PWR0116" (at 69.85 139.7 0)
+    (property "Reference" "#PWR0116" (at 73.66 140.97 0)
       (effects (font (size 1.27 1.27)) hide)
     )
-    (property "Value" "+3.3V" (at 76.9112 140.081 90)
+    (property "Value" "+3.3V" (at 74.041 133.9088 90)
       (effects (font (size 1.27 1.27)) (justify left))
     )
-    (property "Footprint" "" (at 73.66 139.7 0)
+    (property "Footprint" "" (at 73.66 137.16 0)
       (effects (font (size 1.27 1.27)) hide)
     )
-    (property "Datasheet" "" (at 73.66 139.7 0)
+    (property "Datasheet" "" (at 73.66 137.16 0)
       (effects (font (size 1.27 1.27)) hide)
     )
@@
     )
   )
-  (symbol (lib_id "controller-rescue:+3.3V-power") (at 73.66 143.51 270) (unit 1)
-    (in_bom yes) (on_board yes) (dnp no)
-    (property "Reference" "#PWR0117" (at 69.85 143.51 0)
-      (effects (font (size 1.27 1.27)) hide)
-    )
-    (property "Value" "+3.3V" (at 76.9112 143.891 90)
-      (effects (font (size 1.27 1.27)) (justify left))
-    )
-    (property "Footprint" "" (at 73.66 143.51 0)
-      (effects (font (size 1.27 1.27)) hide)
-    )
-    (property "Datasheet" "" (at 73.66 143.51 0)
-      (effects (font (size 1.27 1.27)) hide)
-    )
-    (pin "1")
-    (instances
-      (project "necpc8801typea"
-        (path "/151da08b-0979-4785-a9bf-6fa9b165d629"
-          (reference "#PWR0117") (unit 1)
-        )
-      )
-      (project "controller"
-        (path "/d7b41e20-3ed8-4e20-8d18-95c1ff55bd12"
-          (reference "#PWR0117") (unit 1)
-        )
-      )
-    )
-  )
   (symbol (lib_id "Device:R") (at 64.77 139.7 270) (unit 1)
     (in_bom yes) (on_board yes) (dnp no)
@@
         )
       )
+    )
+  )
+  (symbol (lib_id "controller-rescue:GND-power") (at 73.66 161.29 0) (unit 1)
+    (in_bom yes) (on_board yes) (dnp no)
+    (property "Reference" "#PWR035" (at 73.66 167.64 0)
+      (effects (font (size 1.27 1.27)) hide)
+    )
+    (property "Value" "GND" (at 73.787 165.6842 0)
+      (effects (font (size 1.27 1.27)))
+    )
+    (property "Footprint" "" (at 73.66 161.29 0)
+      (effects (font (size 1.27 1.27)) hide)
+    )
+    (property "Datasheet" "" (at 73.66 161.29 0)
+      (effects (font (size 1.27 1.27)) hide)
+    )
+    (pin "1")
+    (instances
+      (project "necpc8801typea"
+        (path "/151da08b-0979-4785-a9bf-6fa9b165d629"
+          (reference "#PWR035") (unit 1)
+        )
+      )
+      (project "controller"
+        (path "/d7b41e20-3ed8-4e20-8d18-95c1ff55bd12"
+          (reference "#PWR035") (unit 1)
+        )
+      )

Commit message: updates
Connections:
- net COL16: now also U3.23 (PA7); no longer U3.24 (PC4)
- net COL17: now also U3.22 (PA6); no longer U3.23 (PA7)
- net COL18: now also R13.2, U3.21 (PA5); no longer U3.22 (PA6)
- net COL19: now also U3.20 (PA4); no longer R13.2, U3.21 (PA5)
- net ROW3: now also U3.24 (PC4); no longer U3.2 (PC13)
- net ROW5: now also U3.17 (PA3); no longer U3.4 (PC15)
Changed lines of the file:
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@@
   (no_connect (at 58.42 118.745))
   (no_connect (at 125.73 147.32))
-  (no_connect (at 160.02 91.44))
+  (no_connect (at 125.73 160.02))
   (no_connect (at 124.46 121.92))
   (no_connect (at 124.46 124.46))
@@
   (no_connect (at 160.02 114.3))
   (no_connect (at 125.73 157.48))
-  (no_connect (at 160.02 88.9))
+  (no_connect (at 125.73 154.94))
   (no_connect (at 53.34 106.045))
   (wire (pts (xy 107.95 118.11) (xy 104.14 118.11))
@@
     (stroke (width 0) (type solid))
   )
-  (wire (pts (xy 158.75 91.44) (xy 160.02 91.44))
-    (stroke (width 0) (type default))
-  )
   (wire (pts (xy 180.34 129.54) (xy 180.34 139.7))
     (stroke (width 0) (type default))
@@
     (stroke (width 0) (type default))
   )
+  (wire (pts (xy 158.75 91.44) (xy 160.02 91.44))
+    (stroke (width 0) (type default))
+  )
   (wire (pts (xy 31.75 306.07) (xy 34.29 306.07))
     (stroke (width 0) (type solid))
@@
     )
   )
-  (global_label "ROW5" (shape bidirectional) (at 125.73 160.02 180)
-    (effects (font (size 1.27 1.27)) (justify right))
-    (property "Intersheetrefs" "${INTERSHEET_REFS}" (at 125.73 160.02 0)
+  (global_label "ROW5" (shape bidirectional) (at 160.02 88.9 0)
+    (effects (font (size 1.27 1.27)) (justify left))
+    (property "Intersheetrefs" "${INTERSHEET_REFS}" (at 160.02 88.9 0)
       (effects (font (size 1.27 1.27)) hide)
     )
@@
     )
   )
-  (global_label "COL16" (shape bidirectional) (at 124.46 132.08 180)
-    (effects (font (size 1.27 1.27)) (justify right))
-    (property "Intersheetrefs" "${INTERSHEET_REFS}" (at 124.46 132.08 0)
+  (global_label "COL16" (shape bidirectional) (at 160.02 99.06 0)
+    (effects (font (size 1.27 1.27)) (justify left))
+    (property "Intersheetrefs" "${INTERSHEET_REFS}" (at 160.02 99.06 0)
       (effects (font (size 1.27 1.27)) hide)
     )
@@
     )
   )
-  (global_label "COL17" (shape bidirectional) (at 160.02 99.06 0)
+  (global_label "COL17" (shape bidirectional) (at 160.02 96.52 0)
     (effects (font (size 1.27 1.27)) (justify left))
-    (property "Intersheetrefs" "${INTERSHEET_REFS}" (at 160.02 99.06 0)
+    (property "Intersheetrefs" "${INTERSHEET_REFS}" (at 160.02 96.52 0)
       (effects (font (size 1.27 1.27)) hide)
     )
@@
     )
   )
-  (global_label "ROW3" (shape bidirectional) (at 125.73 154.94 180)
+  (global_label "ROW3" (shape bidirectional) (at 124.46 132.08 180)
     (effects (font (size 1.27 1.27)) (justify right))
-    (property "Intersheetrefs" "${INTERSHEET_REFS}" (at 125.73 154.94 0)
+    (property "Intersheetrefs" "${INTERSHEET_REFS}" (at 124.46 132.08 0)
       (effects (font (size 1.27 1.27)) hide)
     )
@@
     )
   )
-  (global_label "COL18" (shape bidirectional) (at 160.02 96.52 0)
+  (global_label "COL18" (shape bidirectional) (at 180.34 93.98 0)
     (effects (font (size 1.27 1.27)) (justify left))
-    (property "Intersheetrefs" "${INTERSHEET_REFS}" (at 160.02 96.52 0)
+    (property "Intersheetrefs" "${INTERSHEET_REFS}" (at 180.34 93.98 0)
       (effects (font (size 1.27 1.27)) hide)
     )
@@
     )
   )
-  (global_label "COL19" (shape bidirectional) (at 180.34 93.98 0)
+  (global_label "COL19" (shape bidirectional) (at 160.02 91.44 0)
     (effects (font (size 1.27 1.27)) (justify left))
-    (property "Intersheetrefs" "${INTERSHEET_REFS}" (at 180.34 93.98 0)
+    (property "Intersheetrefs" "${INTERSHEET_REFS}" (at 160.02 91.44 0)
       (effects (font (size 1.27 1.27)) hide)
     )
@@
   (symbol (lib_id "controller-rescue:GND-power") (at 46.99 128.905 0) (unit 1)
     (in_bom yes) (on_board yes) (dnp no)
-    (property "Reference" "#PWR035" (at 46.99 135.255 0)
+    (property "Reference" "#PWR0105" (at 46.99 135.255 0)
       (effects (font (size 1.27 1.27)) hide)
     )
@@
       (project "necpc8801typea"
         (path "/151da08b-0979-4785-a9bf-6fa9b165d629"
-          (reference "#PWR035") (unit 1)
+          (reference "#PWR0105") (unit 1)
         )
       )

Commit message: updates
Parts:
- removed J1: Conn_01x01, Connector_PinHeader_1.27mm:PinHeader_1x01_P1.27mm_Vertical, symbol controller-rescue:Conn_01x01-Connector_Generic
- removed J2: Conn_01x06, Connector_PinHeader_1.27mm:PinHeader_1x06_P1.27mm_Vertical, symbol controller-rescue:Conn_01x06-Connector_Generic
Changed lines of the file:
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@@
-    )
-  )
-  (symbol (lib_id "controller-rescue:Conn_01x06-Connector_Generic") (at 231.14 55.88 0) (unit 1)
-    (in_bom yes) (on_board yes) (dnp no)
-    (property "Reference" "J2" (at 233.172 56.0832 0)
-      (effects (font (size 1.27 1.27)) (justify left))
-    )
-    (property "Value" "Conn_01x06" (at 233.172 58.3946 0)
-      (effects (font (size 1.27 1.27)) (justify left))
-    )
-    (property "Footprint" "Connector_PinHeader_1.27mm:PinHeader_1x06_P1.27mm_Vertical" (at 231.14 55.88 0)
-      (effects (font (size 1.27 1.27)) hide)
-    )
-    (property "Datasheet" "~" (at 231.14 55.88 0)
-      (effects (font (size 1.27 1.27)) hide)
-    )
-    (pin "1")
-    (pin "2")
-    (pin "3")
-    (pin "4")
-    (pin "5")
-    (pin "6")
-    (instances
-      (project "necpc8801typea"
-        (path "/151da08b-0979-4785-a9bf-6fa9b165d629"
-          (reference "J2") (unit 1)
-        )
-      )
-      (project "controller"
-        (path "/d7b41e20-3ed8-4e20-8d18-95c1ff55bd12"
-          (reference "J6") (unit 1)
-        )
-      )
     )
   )
@@
     )
   )
-  (symbol (lib_id "controller-rescue:Conn_01x01-Connector_Generic") (at 231.14 44.45 0) (unit 1)
-    (in_bom yes) (on_board yes) (dnp no)
-    (property "Reference" "J1" (at 233.172 43.3832 0)
-      (effects (font (size 1.27 1.27)) (justify left))
-    )
-    (property "Value" "Conn_01x01" (at 233.172 45.6946 0)
-      (effects (font (size 1.27 1.27)) (justify left))
-    )
-    (property "Footprint" "Connector_PinHeader_1.27mm:PinHeader_1x01_P1.27mm_Vertical" (at 231.14 44.45 0)
-      (effects (font (size 1.27 1.27)) hide)
-    )
-    (property "Datasheet" "~" (at 231.14 44.45 0)
-      (effects (font (size 1.27 1.27)) hide)
-    )
-    (pin "1")
-    (instances
-      (project "necpc8801typea"
-        (path "/151da08b-0979-4785-a9bf-6fa9b165d629"
-          (reference "J1") (unit 1)
-        )
-      )
-      (project "controller"
-        (path "/d7b41e20-3ed8-4e20-8d18-95c1ff55bd12"
-          (reference "J4") (unit 1)
-        )
-      )
-    )
-  )
   (symbol (lib_id "Device:Q_NMOS_GSD") (at 30.48 102.235 0) (mirror y) (unit 1)
     (in_bom yes) (on_board yes) (dnp no)
@@
         )
       )
-    )
-  )
-  (symbol (lib_id "controller-rescue:+3.3V-power") (at 226.06 44.45 90) (unit 1)
-    (in_bom yes) (on_board yes) (dnp no)
-    (property "Reference" "#PWR0119" (at 229.87 44.45 0)
-      (effects (font (size 1.27 1.27)) hide)
-    )
-    (property "Value" "+3.3V" (at 222.8088 44.069 90)
-      (effects (font (size 1.27 1.27)) (justify left))
-    )
-    (property "Footprint" "" (at 226.06 44.45 0)
-      (effects (font (size 1.27 1.27)) hide)
-    )
-    (property "Datasheet" "" (at 226.06 44.45 0)
-      (effects (font (size 1.27 1.27)) hide)
-    )
-    (pin "1")
-    (instances
-      (project "necpc8801typea"
-        (path "/151da08b-0979-4785-a9bf-6fa9b165d629"
-          (reference "#PWR0119") (unit 1)
-        )
-      )
-      (project "controller"
-        (path "/d7b41e20-3ed8-4e20-8d18-95c1ff55bd12"
-          (reference "#PWR0119") (unit 1)
-        )
-      )

Commit message: updates
Parts:
- removed J4: Conn_01x04, Connector_JST:JST_PH_S4B-PH-K_1x04_P2.00mm_Horizontal, symbol controller-rescue:Conn_01x04-Connector_Generic
- added J2: Conn_01x04_MountingPin, Connector_JST:JST_SH_SM04B-SRSS-TB_1x04-1MP_P1.00mm_Horizontal, symbol Connector_Generic_MountingPin:Conn_01x04_MountingPin
- added Q4: 2N3904, Package_TO_SOT_SMD:SOT-23, symbol Transistor_BJT:2N3904
- R4: value 22 -> 1k
Connections:
- net GPIO_PB3 is gone; now on an unnamed net: U3.55 (PB3)
- net +5V: now also BUZ1.1, C21.1
- net BUZIN: now also R4.2, U3.20 (PA4); no longer R4.1
- net COL19: now also U3.46 (PA13); no longer U3.20 (PA4)
- net GND: now also J2.1 (Pin_1), Q4.1 (E); no longer BUZ1.2
- net USB_DM_ESD: now also J2.3 (Pin_3)
- net USB_DP_ESD: now also J2.2 (Pin_2)
- net VBUS: now also J2.4 (Pin_4)
- new net: BUZ1.2, Q4.3 (C)
- new net: Q4.2 (B), R4.1
- no-connect marks 16 -> 14
Other:
- moved on the sheet: BUZ1, C21, R4, R6

Commit message: change crystal setup
Parts:
- removed R7: 390, Resistor_SMD:R_0805_2012Metric_Pad1.20x1.40mm_HandSolder, symbol Device:R
- Y1: value 16MHz -> 8MHz; footprint Crystal:Crystal_SMD_3225-4Pin_3.2x2.5mm_HandSoldering -> acheron_Components:Crystal_SMD_3225-4Pin_3.2x2.5mm; LCSC C13738 -> C389817
Connections:
- net OSCO_RES is gone; now on net OSCO: C24.1, Y1.3
Changed lines of the file:
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@@
   (no_connect (at 125.73 154.94))
   (no_connect (at 53.34 106.045))
-  (wire (pts (xy 107.95 118.11) (xy 104.14 118.11))
+  (wire (pts (xy 88.9 118.11) (xy 107.95 118.11))
     (stroke (width 0) (type default))
   )
@@
     (stroke (width 0) (type solid))
   )
-  (wire (pts (xy 88.9 118.11) (xy 96.52 118.11))
-    (stroke (width 0) (type default))
-  )
   (wire (pts (xy 66.04 325.12) (xy 68.58 325.12))
     (stroke (width 0) (type solid))
@@
     )
   )
-  (symbol (lib_id "Device:R") (at 100.33 118.11 90) (unit 1)
-    (in_bom yes) (on_board yes) (dnp no)
-    (property "Reference" "R7" (at 99.06 120.65 90)
-      (effects (font (size 1.27 1.27)))
-    )
-    (property "Value" "390" (at 102.87 120.65 90)
-      (effects (font (size 1.27 1.27)))
-    )
-    (property "Footprint" "Resistor_SMD:R_0805_2012Metric_Pad1.20x1.40mm_HandSolder" (at 100.33 119.888 90)
-      (effects (font (size 1.27 1.27)) hide)
-    )
-    (property "Datasheet" "~" (at 100.33 118.11 0)
-      (effects (font (size 1.27 1.27)) hide)
-    )
-    (property "LCSC" "C17655" (at 100.33 118.11 0)
-      (effects (font (size 1.27 1.27)) hide)
-    )
-    (pin "1")
-    (pin "2")
-    (instances
-      (project "necpc8801typea"
-        (path "/151da08b-0979-4785-a9bf-6fa9b165d629"
-          (reference "R7") (unit 1)
-        )
-      )
-      (project "controller"
-        (path "/d7b41e20-3ed8-4e20-8d18-95c1ff55bd12"
-          (reference "R1") (unit 1)
-        )
-      )
-    )
-  )
   (symbol (lib_id "Device:R") (at 64.77 151.13 270) (unit 1)
     (in_bom yes) (on_board yes) (dnp no)
@@
       (effects (font (size 1.27 1.27)) (justify left))
     )
-    (property "Value" "16MHz" (at 94.615 109.855 90)
+    (property "Value" "8MHz" (at 94.615 109.855 90)
       (effects (font (size 1.27 1.27)) (justify left))
     )
-    (property "Footprint" "Crystal:Crystal_SMD_3225-4Pin_3.2x2.5mm_HandSoldering" (at 88.9 110.49 0)
+    (property "Footprint" "acheron_Components:Crystal_SMD_3225-4Pin_3.2x2.5mm" (at 88.9 110.49 0)
       (effects (font (size 1.27 1.27)) hide)
     )
-    (property "Datasheet" "https://datasheet.lcsc.com/szlcsc/Yangxing-Tech-X322516MLB4SI_C13738.pdf" (at 88.9 110.49 0)
+    (property "Datasheet" "https://datasheet.lcsc.com/lcsc/1912111437_XTY-7325-0800A2010-00_C389817.pdf" (at 88.9 110.49 0)
       (effects (font (size 1.27 1.27)) hide)
     )
-    (property "LCSC" "C13738" (at 88.9 110.49 90)
+    (property "LCSC" "C389817" (at 88.9 110.49 90)
       (effects (font (size 1.27 1.27)) hide)
     )

Commit message: cleanup
Connections:
- net COL16: now also U3.22 (PA6); no longer U3.23 (PA7)
- net COL17: now also R13.2, U3.21 (PA5); no longer U3.22 (PA6)
- net COL18: now also U3.46 (PA13); no longer R13.2, U3.21 (PA5)
- net COL19: now also U3.17 (PA3); no longer U3.46 (PA13)
- net ROW3: now also U3.23 (PA7); no longer U3.24 (PC4)
- net ROW5: now also U3.24 (PC4); no longer U3.17 (PA3)

Commit message: updates
Parts:
- removed C4, C5, C7: 100nF, Capacitor_SMD:C_0805_2012Metric_Pad1.18x1.45mm_HandSolder, symbol Device:C
- removed C6, C9: 22uF, Capacitor_SMD:C_0805_2012Metric_Pad1.18x1.45mm_HandSolder, symbol Device:C
- removed R1, R13: 62k, Resistor_SMD:R_0805_2012Metric_Pad1.20x1.40mm_HandSolder, symbol Device:R
- removed U2: TPS2553DBVR, Package_TO_SOT_SMD:SOT-23-6_Handsoldering, symbol tps2553dbvr:TPS2553DBVR
- added R18, R19: 62k, Resistor_SMD:R_0805_2012Metric_Pad1.20x1.40mm_HandSolder, symbol Device:R
- C8: value 100nF -> 1uF
- U1: value AMS1117-3.3 -> XC6206P332NR
Connections:
- net +3.3VA: now also R16.1, R17.1, R18.1, R19.1
- net +5V: now also C3.1, FB1.1
- net COL1: now also R12.2; no longer R15.2
- net COL10: now also R18.2
- net COL12: no longer R17.2
- net COL17: now also R17.2
- net COL4: no longer R12.2
- net COL6: no longer R14.2
- net EEP_SCL: now also U3.61 (PB8); no longer U3.15 (PA1)
- net EEP_SDA: now also U3.62 (PB9); no longer U3.16 (PA2)
- net GND: no longer R16.1, R17.1, U3.58 (PB6), U3.62 (PB9)
- net ROW0: now also U3.24 (PC4); no longer U3.61 (PB8)
- net ROW5: now also U3.15 (PA1); no longer U3.24 (PC4)
- net PB3: now reaches R6.2, U3.55 (PB3)
- net PB3: now also R15.2
- net PC10: now reaches U3.51 (PC10)
- net PC10: now also R19.2
- net PB4: now reaches U3.56 (PB4)
- net PB4: now also R16.2
- net PB7: now reaches U3.59 (PB7)
- net PB7: now also R14.2
- net PC11 renamed ROW1
- net ROW1: no longer R16.2
Other:
- note added: "These are all pulled up to disable all non-DFU bootloader modes"
- moved on the sheet: BUZ1, C16, C17, C18, C21, C3, C8, LED1, LED2, LED3, Q4, R10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
