File: necpc8801typea.kicad_sch (KiCad schematic)
At the start: 257 parts, among them J2 Conn_01x04_MountingPin, Q1 Q_PMOS_GSD AO3401A, Q2 Q_NMOS_GSD 2N7002, Q3 Q_NMOS_GSD 2N7002, Q4 2N3904, SW1 SW_Push, U1 XC6206P332NR, U3 STM32F401RETx, U4 24LC64, U5 USBLC6-2SC6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

Commit message: updates
Parts:
- added U2: 74AHCT1G125, Package_TO_SOT_SMD:SOT-23-5, symbol 74xGxx:74AHCT1G125
Connections:
- net +5V: now also U2.5 (VCC)
- net GND: now also U2.1, U2.3 (GND)
- net LEDDIN: now also U2.2; no longer LED3.4 (DIN), R6.1
- new net LEDDINC: LED3.4 (DIN), U2.4
Other:
- moved on the sheet: C16, C17, C18, LED1, LED2, LED3
